File: cc-component.kicad_sch (KiCad schematic)
At the start: 36 parts, among them J201 B-057-HP, J202 2227MC-06-03, J203 B-057-HP, J204 B-057-HP, Q201 SSM6L56FE, U201 OPA2333AIDR, U202 REF35102QDBVR

Commit message: feat: v1.1 として現行版の定電流回路を取り込む
HVRF リポジトリの作業ツリー（2026-10-15 時点）を v1.1 として取り込む。

- プロジェクトを transistor-hfe-measurement-circuit に改名
  （サブシートは cc-component.kicad_sch）
- 回路図・PCB のタイトルブロックに版数・著作権・ライセンス
  （CERN-OHL-P v2）・リポジトリ URL を入れる
- 基板シルクの版数を V1.0 から V1.1 にする
- PCB にはメーカー製 3D モデルを埋め込まず、DC ジャックは自作の
  簡易モデルを参照する

Co-Authored-By: Claude Opus 5.5 <noreply@anthropic.com>
Other:
- company: (none) -> Hayata Yamamoto
- title: (none) -> Transistor hFE Measurement Circuit Schematic
